File: Accumulator.kicad_sch (KiCad schematic)
At the start: 31 parts, among them J6 1988817, J7 1190363, J8 1190363, K1 AWHSH105D00G, K2 AWHSH105D00G, Q7 GT065P06T, Q8 IRFZ44N, U4 UCC37324P, U8 ULN2003, U9 MCP4151-xxxx-P

Commit message: Reviewed gate resistors and removed MOSFET driver resistor
Parts:
- removed R15: 47Ω, Resistor_THT:R_Axial_DIN0207_L6.3mm_D2.5mm_P10.16mm_Horizontal, symbol Device:R_US
- added TP14: TestPoint, TestPoint:TestPoint_THTPad_1.0x1.0mm_Drill0.5mm, symbol Connector:TestPoint
Connections:
- net RELAYS: now also TP14.1
- net at U4.7 (OUTA): now also Q8.1 (G), TP31.1
Other:
- note added: "Defiently not needed, but was cool to learn about."
- moved on the sheet: TP31
Changed lines of the file:
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@@
 	)
 	(junction
-		(at 241.3 138.43)
-		(diameter 0)
-		(color 0 0 0 0)
-	)
-	(junction
 		(at 91.44 27.94)
 		(diameter 0)
@@
 	)
 	(junction
+		(at 233.68 138.43)
+		(diameter 0)
+		(color 0 0 0 0)
+	)
+	(junction
 		(at 53.34 21.59)
 		(diameter 0)
@@
 	(wire
 		(pts
-			(xy 223.52 138.43) (xy 229.87 138.43)
+			(xy 223.52 138.43) (xy 233.68 138.43)
 		)
 		(stroke
@@
 	(wire
 		(pts
-			(xy 237.49 138.43) (xy 241.3 138.43)
-		)
-		(stroke
-			(width 0)
-			(type default)
-		)
-	)
-	(wire
-		(pts
 			(xy 59.69 134.62) (xy 59.69 138.43)
 		)
@@
 	(wire
 		(pts
-			(xy 43.18 85.09) (xy 50.8 85.09)
+			(xy 233.68 138.43) (xy 247.65 138.43)
 		)
 		(stroke
@@
 	(wire
 		(pts
-			(xy 241.3 138.43) (xy 247.65 138.43)
+			(xy 43.18 85.09) (xy 50.8 85.09)
 		)
 		(stroke
@@
 		)
 	)
+	(text "Defiently not needed, but was cool to learn about.\n"
+		(exclude_from_sim no)
+		(at 204.724 160.528 0)
+		(effects
+			(font
+				(size 1.27 1.27)
+			)
+		)
+	)
 	(text "9091Ω in when parallel, 3704Ω when in series"
 		(exclude_from_sim no)
@@
 	)
 	(symbol
+		(lib_id "Connector:TestPoint")
+		(at 97.79 72.39 0)
+		(unit 1)
+		(exclude_from_sim no)
+		(in_bom yes)
+		(on_board yes)
+		(dnp no)
+		(property "Reference" "TP14"
+			(at 95.504 66.802 0)
+			(effects
+				(font
+					(size 1.27 1.27)
+				)
+				(justify left)
+			)
+		)
+		(property "Value" "TestPoint"
+			(at 100.33 70.3579 0)
+			(effects
+				(font
+					(size 1.27 1.27)
+				)
+				(justify left)
+				(hide yes)
+			)
+		)
+		(property "Footprint" "TestPoint:TestPoint_THTPad_1.0x1.0mm_Drill0.5mm"
+			(at 102.87 72.39 0)
+			(effects
+				(font
+					(size 1.27 1.27)
+				)
+				(hide yes)
+			)
+		)
+		(property "Datasheet" "~"
+			(at 102.87 72.39 0)
+			(effects
+				(font
+					(size 1.27 1.27)
+				)
+				(hide yes)
+			)
+		)
+		(property "Description" "test point"
+			(at 97.79 72.39 0)
+			(effects
+				(font
+					(size 1.27 1.27)
+				)
+				(hide yes)
+			)
+		)
+		(pin "1"
+		)
+		(instances
+			(project "SuperCapacitorBike"
+				(path "/1096cbe7-ac56-48cb-aadd-3e4addcdbbb7/a3002b5e-253f-453a-a6f1-d0dba20d26d3"
+					(reference "TP14")
+					(unit 1)
+				)
+			)
+		)
+	)
+	(symbol
 		(lib_id "power:GND")
 		(at 259.08 22.86 0)
@@
 	)
 	(symbol
-		(lib_id "Device:R_US")
-		(at 233.68 138.43 90)
-		(unit 1)
-		(exclude_from_sim no)
-		(in_bom yes)
-		(on_board yes)
-		(dnp no)
-		(fields_autoplaced yes)
-		(property "Reference" "R15"
-			(at 233.68 132.08 90)
-			(effects
-				(font
-					(size 1.27 1.27)
-				)
-			)
-		)
-		(property "Value" "47Ω"
-			(at 233.68 134.62 90)
-			(effects
-				(font
-					(size 1.27 1.27)
-				)
-			)
-		)
-		(property "Footprint" "Resistor_THT:R_Axial_DIN0207_L6.3mm_D2.5mm_P10.16mm_Horizontal"
-			(at 233.934 137.414 90)
-			(effects
-				(font
-					(size 1.27 1.27)
-				)
-				(hide yes)
-			)
-		)
-		(property "Datasheet" "~"
-			(at 233.68 138.43 0)
-			(effects
-				(font
-					(size 1.27 1.27)
-				)
-				(hide yes)
-			)
-		)
-		(property "Description" "Resistor, US symbol"
-			(at 233.68 138.43 0)
-			(effects
-				(font
-					(size 1.27 1.27)
-				)
-				(hide yes)
-			)
-		)
-		(pin "1"
-		)
-		(pin "2"
-		)
-		(instances
-			(project ""
-				(path "/1096cbe7-ac56-48cb-aadd-3e4addcdbbb7/a3002b5e-253f-453a-a6f1-d0dba20d26d3"
-					(reference "R15")
-					(unit 1)
-				)
-			)
-		)
-	)
-	(symbol
 		(lib_id "Mechanical:MountingHole_Pad")
 		(at 259.08 20.32 0)
@@
 	(symbol
 		(lib_id "Connector:TestPoint")
-		(at 241.3 138.43 0)
+		(at 233.68 138.43 0)
 		(unit 1)
 		(exclude_from_sim no)
@@
 		(dnp no)
 		(property "Reference" "TP31"
-			(at 239.014 133.35 0)
+			(at 231.394 133.35 0)
 			(effects
 				(font
@@
 		)
 		(property "Value" "TestPoint"
-			(at 243.84 136.3979 0)
+			(at 236.22 136.3979 0)
 			(effects
 				(font
@@
 		)
 		(property "Footprint" "TestPoint:TestPoint_THTPad_1.0x1.0mm_Drill0.5mm"
-			(at 246.38 138.43 0)
+			(at 238.76 138.43 0)
 			(effects
 				(font
@@
 		)
 		(property "Datasheet" "~"
-			(at 246.38 138.43 0)
+			(at 238.76 138.43 0)
 			(effects
 				(font
@@
 		)
 		(property "Description" "test point"
-			(at 241.3 138.43 0)
+			(at 233.68 138.43 0)
 			(effects
 				(font

Commit message: Prototyping PCB Ordered!
Parts:
- added R2: 0Ω, Resistor_THT:R_Axial_DIN0207_L6.3mm_D2.5mm_P10.16mm_Horizontal, symbol Device:R_US
- added TP15: TestPoint, TestPoint:TestPoint_THTPad_1.0x1.0mm_Drill0.5mm, symbol Connector:TestPoint
Connections:
- net C1+: now also TP31.1
- new net: R2.1, U4.7 (OUTA)
- new net: Q8.1 (G), R2.2, TP15.1
Other:
- note added: "Although I am not super focused on reducing EMI, I am still interested in learning how to mitagate when switching MOSFETS: Because the trace is so long, there is likely a non-negligible amount of parasitic inductance and capacitance resulting in a %OS that I can not emperically measure. I put a 0Ω resistor in hopes I can sweet talk the lab techs to let me use their good DSO's and test =)"
- moved on the sheet: K1, K2, TP14, TP24, TP25, TP30, TP33, U8

Commit message: Changed voltage divider resistors
Parts:
- R16: value 20kΩ -> 22kΩ
- R17: value 55kΩ -> 22kΩ
- R18: value 25kΩ -> 10kΩ
Other:
- note added: "10kΩ in when parallel, 4074Ω when in series"
- note removed: "9091Ω in when parallel, 3704Ω when in series"
Changed lines of the file:
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@@
 		)
 	)
-	(text "9091Ω in when parallel, 3704Ω when in series"
+	(text "10kΩ in when parallel, 4074Ω when in series"
 		(exclude_from_sim no)
 		(at 44.45 110.49 0)
@@
 			)
 		)
-		(property "Value" "25kΩ"
+		(property "Value" "10kΩ"
 			(at 45.72 93.9799 0)
 			(effects
@@
 			)
 		)
-		(property "Value" "20kΩ"
+		(property "Value" "22kΩ"
 			(at 62.23 128.2699 0)
 			(effects
@@
 			)
 		)
-		(property "Value" "55kΩ"
+		(property "Value" "22kΩ"
 			(at 45.72 78.7399 0)
 			(effects
